File: KiCad_PDM/Gate_driver.kicad_sch (KiCad schematic)
At the start: 25 parts, among them U10 INA180A3IDBVR, U6 2N7002, U7 NSG2000, U8 OSP80N03T, U9 2N7002

Commit message: updated design and 3d models
Parts:
- added D6: 1N5819HW-7-F, Diode_SMD:D_SOD-123, symbol PDM:DIODES 1N5819HW-7-F
- renumbered D6 to D7, D7 to D8
Connections:
- net GND: now also D6.2 (A)
- net at C10.2, D3.2, D5.2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: now also D6.1 (K)
