File: KiCad_PDM/KiCad_PDM.kicad_pcb (KiCad board)
At the start: 4 copper layers, 100 x 175 mm, 327 parts, among them J1 Conn_02x16_Top_Bottom, J2 6437288-1, J3 T66145145-1500, U1 74HC27D, U10 INA180A3IDBVR, U11 2N7002, U12 NSG2000, U13 OSP80N03T, U14 2N7002, U15 INA180A3IDBVR, U16 2N7002, U17 NSG2000, U18 OSP80N03T, U19 2N7002, U2 74HC27D, U20 INA180A3IDBVR, U21 2N7002, U22 NSG2000, U23 OSP80N03T, U24 2N7002, U25 INA180A3IDBVR, U26 2N7002, U27 NSG2000, U28 OSP80N03T, U29 2N7002, U3 74HC27D, U30 INA180A3IDBVR, U31 2N7002, U32 NSG2000, U33 OSP80N03T, U34 2N7002, U35 INA180A3IDBVR, U36 2N7002, U37 NSG2000, U38 OSP80N03T, U39 2N7002, U4 74HC27D, U40 INA180A3IDBVR, U41 2N7002, U42 NSG2000, U43 OSP80N03T, U44 2N7002, U45 INA180A3IDBVR, U46 2N7002, U47 NSG2000, U48 OSP80N03T, U49 2N7002, U5 KF33BDT-TR, U50 INA180A3IDBVR, U51 2N7002, U52 NSG2000, U53 OSP80N03T, U54 2N7002, U55 INA180A3IDBVR, U6 2N7002, U7 NSG2000, U8 OSP80N03T, U9 2N7002

Commit message: Added TS/Souce connections, fixed flyback diode connections, fixed current sense kelvin connections
Parts:
- added C57: C_Polarized, Capacitor_THT:CP_Radial_D8.0mm_P2.50mm, F.Cu at (60.4, 79.0)
- added C58: C_Polarized, Capacitor_THT:CP_Radial_D8.0mm_P2.50mm, F.Cu at (60.4, 120.1)
- turned D15 to 0 degrees
- turned D22 to 0 degrees
- turned D29 to 0 degrees
- turned D36 to 0 degrees
- turned D43 to 0 degrees
- turned D50 to 0 degrees
- turned D57 to 0 degrees
- turned D64 to 0 degrees
- turned D71 to 0 degrees
- turned D8 to 0 degrees
Connections:
- D15 pad 1: +BATT -> Net-(D13-K)
- D15 pad 2: Net-(U13-Source) -> GND
- D22 pad 1: +BATT -> Net-(D20-K)
- D22 pad 2: Net-(U18-Source) -> GND
- D29 pad 1: +BATT -> Net-(D27-K)
- D29 pad 2: Net-(U23-Source) -> GND
- D36 pad 1: +BATT -> Net-(D34-K)
- D36 pad 2: Net-(U28-Source) -> GND
- D43 pad 1: +BATT -> Net-(D41-K)
- D43 pad 2: Net-(U33-Source) -> GND
- D50 pad 1: +BATT -> Net-(D48-K)
- D50 pad 2: Net-(U38-Source) -> GND
- D57 pad 1: +BATT -> Net-(D55-K)
- D57 pad 2: Net-(U43-Source) -> GND
- D64 pad 1: +BATT -> Net-(D62-K)
- D64 pad 2: Net-(U48-Source) -> GND
- D71 pad 1: +BATT -> Net-(D69-K)
- D71 pad 2: Net-(U53-Source) -> GND
- D8 pad 1: +BATT -> Net-(D6-K)
- D8 pad 2: Net-(U10-In+) -> GND
- R106 pad 1: Net-(U48-Source) -> Net-(D62-K)
- R115 pad 1: Net-(U53-Source) -> Net-(D69-K)
- R34 pad 1: Net-(U10-In+) -> Net-(D6-K)
- R43 pad 1: Net-(U13-Source) -> Net-(D13-K)
- R52 pad 1: Net-(U18-Source) -> Net-(D20-K)
- R61 pad 1: Net-(U23-Source) -> Net-(D27-K)
- R70 pad 1: Net-(U28-Source) -> Net-(D34-K)
- R79 pad 1: Net-(U33-Source) -> Net-(D41-K)
- R88 pad 1: Net-(U38-Source) -> Net-(D48-K)
- R97 pad 1: Net-(U43-Source) -> Net-(D55-K)
- U10 pad 3: Net-(U10-In+) -> Net-(D6-K)
- U13 pad 3: Net-(U13-Source) -> Net-(D13-K)
- U14 pad 1: Net-(U13-Source) -> Net-(D13-K)
- U15 pad 3: Net-(U13-Source) -> Net-(D13-K)
- U18 pad 3: Net-(U18-Source) -> Net-(D20-K)
- U19 pad 1: Net-(U18-Source) -> Net-(D20-K)
- U20 pad 3: Net-(U18-Source) -> Net-(D20-K)
- U23 pad 3: Net-(U23-Source) -> Net-(D27-K)
- U24 pad 1: Net-(U23-Source) -> Net-(D27-K)
- U25 pad 3: Net-(U23-Source) -> Net-(D27-K)
- U28 pad 3: Net-(U28-Source) -> Net-(D34-K)
- U29 pad 1: Net-(U28-Source) -> Net-(D34-K)
- U30 pad 3: Net-(U28-Source) -> Net-(D34-K)
- U33 pad 3: Net-(U33-Source) -> Net-(D41-K)
- U34 pad 1: Net-(U33-Source) -> Net-(D41-K)
- U35 pad 3: Net-(U33-Source) -> Net-(D41-K)
- U38 pad 3: Net-(U38-Source) -> Net-(D48-K)
- U39 pad 1: Net-(U38-Source) -> Net-(D48-K)
- U40 pad 3: Net-(U38-Source) -> Net-(D48-K)
- U43 pad 3: Net-(U43-Source) -> Net-(D55-K)
- U44 pad 1: Net-(U43-Source) -> Net-(D55-K)
- U45 pad 3: Net-(U43-Source) -> Net-(D55-K)
- U48 pad 3: Net-(U48-Source) -> Net-(D62-K)
- U49 pad 1: Net-(U48-Source) -> Net-(D62-K)
- U50 pad 3: Net-(U48-Source) -> Net-(D62-K)
- U53 pad 3: Net-(U53-Source) -> Net-(D69-K)
- U54 pad 1: Net-(U53-Source) -> Net-(D69-K)
- U55 pad 3: Net-(U53-Source) -> Net-(D69-K)
- U8 pad 3: Net-(U10-In+) -> Net-(D6-K)
- U9 pad 1: Net-(U10-In+) -> Net-(D6-K)
Routing:
- net +BATT: track 304.5 -> 250.7 mm, vias 0 -> 36
- net Net-(D69-K): track 18.2 -> 43.5 mm
- net Net-(D27-K): track 18.2 -> 43.3 mm, vias 2 -> 3
- net Net-(D20-K): track 18.2 -> 43.1 mm, vias 2 -> 3
- net Net-(D48-K): track 18.2 -> 42.9 mm, vias 2 -> 3
- net Net-(D62-K): track 18.2 -> 42.9 mm
- net Net-(D6-K): track 18.7 -> 43.2 mm, vias 2 -> 3
- net Net-(D34-K): track 18.2 -> 42.4 mm, vias 2 -> 3
- net Net-(D55-K): track 22.3 -> 45.8 mm, vias 2 -> 3
- net Net-(D13-K): track 18.2 -> 41.7 mm, vias 2 -> 3
- net Net-(D41-K): track 19.3 -> 41.8 mm, vias 2 -> 3
- net Net-(U43-Source): track 13.3 -> 0.00 mm, vias 1 -> 0
- net Net-(U23-Source): track 13.3 -> 0.00 mm, vias 1 -> 0
- net Net-(U18-Source): track 13.3 -> 0.00 mm, vias 1 -> 0
- net Net-(U13-Source): track 13.3 -> 0.00 mm, vias 1 -> 0
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- added copper zone on B.Cu, net +BATT
