File: KiCad_PDM/KiCad_PDM.kicad_pcb (KiCad board)
At the start: 4 copper layers, 100 x 175 mm, 329 parts, among them J1 Conn_02x16_Top_Bottom, J2 6437288-1, J3 T66145145-1500, U1 74HC27D, U10 INA180A3IDBVR, U11 2N7002, U12 NSG2000, U13 OSP80N03T, U14 2N7002, U15 INA180A3IDBVR, U16 2N7002, U17 NSG2000, U18 OSP80N03T, U19 2N7002, U2 74HC27D, U20 INA180A3IDBVR, U21 2N7002, U22 NSG2000, U23 OSP80N03T, U24 2N7002, U25 INA180A3IDBVR, U26 2N7002, U27 NSG2000, U28 OSP80N03T, U29 2N7002, U3 74HC27D, U30 INA180A3IDBVR, U31 2N7002, U32 NSG2000, U33 OSP80N03T, U34 2N7002, U35 INA180A3IDBVR, U36 2N7002, U37 NSG2000, U38 OSP80N03T, U39 2N7002, U4 74HC27D, U40 INA180A3IDBVR, U41 2N7002, U42 NSG2000, U43 OSP80N03T, U44 2N7002, U45 INA180A3IDBVR, U46 2N7002, U47 NSG2000, U48 OSP80N03T, U49 2N7002, U5 KF33BDT-TR, U50 INA180A3IDBVR, U51 2N7002, U52 NSG2000, U53 OSP80N03T, U54 2N7002, U55 INA180A3IDBVR, U6 2N7002, U7 NSG2000, U8 OSP80N03T, U9 2N7002

Commit message: added production files (gerbers, BOM, 3D models)
Parts:
- C57, C58: value C_Polarized -> 470uF
Changed lines of the file:
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@@
 			)
 		)
-		(property "Value" "C_Polarized"
+		(property "Value" "470uF"
 			(at 1.25 5.25 0)
 			(layer "F.Fab")
@@
 			(pinfunction "GND_2")
 			(pintype "power_in")
+			(zone_connect 2)
 		)
 		(pad "3" smd roundrect
@@
 			)
 		)
-		(property "Value" "C_Polarized"
+		(property "Value" "470uF"
 			(at 1.25 5.25 0)
 			(layer "F.Fab")

Commit message: fixed diff pair trace width -> 0.12mm
Routing:
- net CAN-: track 78.0 -> 77.4 mm
Changed lines of the file:
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@@
 		(capping no)
 		(filling no)
+		(zone_defaults)
 		(pcbplotparams
 			(layerselection 0x00000000_00000000_55555555_5755f5ff)
@@
 	)
 	(segment
-		(start 53.925 98.5)
-		(end 53.934586 98.490414)
-		(width 0.2)
-		(layer "In1.Cu")
-		(net "CAN+")
-	)
-	(segment
 		(start 129.44 99)
 		(end 129.71 98.73)
-		(width 0.2)
-		(layer "In1.Cu")
-		(net "CAN+")
-	)
-	(segment
-		(start 53.929051 98.495949)
-		(end 57.245949 98.495949)
-		(width 0.2)
+		(width 0.12)
 		(layer "In1.Cu")
 		(net "CAN+")
 	)
 	(segment
-		(start 58.5 99.75)
-		(end 82.646446 99.75)
-		(width 0.2)
-		(layer "In1.Cu")
-		(net "CAN+")
-	)
-	(segment
-		(start 57.245949 98.495949)
-		(end 58.5 99.75)
-		(width 0.2)
+		(start 53.925 98.5)
+		(end 57.5 98.5)
+		(width 0.12)
 		(layer "In1.Cu")
 		(net "CAN+")
 	)
 	(segment
-		(start 53.925 98.5)
-		(end 53.929051 98.495949)
-		(width 0.2)
+		(start 57.5 98.5)
+		(end 58.79 99.79)
+		(width 0.12)
 		(layer "In1.Cu")
 		(net "CAN+")
 	)
 	(segment
-		(start 83.396446 99)
+		(start 83.953014 99)
 		(end 129.44 99)
-		(width 0.2)
+		(width 0.12)
 		(layer "In1.Cu")
 		(net "CAN+")
 	)
 	(segment
-		(start 82.646446 99.75)
-		(end 83.396446 99)
-		(width 0.2)
+		(start 83.163014 99.79)
+		(end 83.953014 99)
+		(width 0.12)
 		(layer "In1.Cu")
 		(net "CAN+")
 	)
 	(segment
-		(start 53.928883 101.503883)
-		(end 57.230492 101.503883)
-		(width 0.2)
-		(layer "In1.Cu")
-		(net "CAN-")
-	)
-	(segment
-		(start 58.484375 100.25)
-		(end 82.853554 100.25)
-		(width 0.2)
+		(start 58.79 99.79)
+		(end 83.163014 99.79)
+		(width 0.12)
 		(layer "In1.Cu")
-		(net "CAN-")
+		(net "CAN+")
 	)
 	(segment
-		(start 53.925 101.5)
-		(end 53.934789 101.490211)
-		(width 0.2)
+		(start 84.126986 99.42)
+		(end 127.86 99.42)
+		(width 0.12)
 		(layer "In1.Cu")
 		(net "CAN-")
 	)
 	(segment
-		(start 127.94 99.5)
-		(end 129.71 101.27)
-		(width 0.2)
+		(start 58.79 100.21)
+		(end 83.336986 100.21)
+		(width 0.12)
 		(layer "In1.Cu")
 		(net "CAN-")
@@
 	(segment
 		(start 53.925 101.5)
-		(end 53.928883 101.503883)
-		(width 0.2)
+		(end 57.5 101.5)
+		(width 0.12)
 		(layer "In1.Cu")
 		(net "CAN-")
 	)
 	(segment
-		(start 129.71 101.27)
-		(end 129.23 101.75)
-		(width 0.2)
+		(start 57.5 101.5)
+		(end 58.79 100.21)
+		(width 0.12)
 		(layer "In1.Cu")
 		(net "CAN-")
 	)
 	(segment
-		(start 82.853554 100.25)
-		(end 83.603554 99.5)
-		(width 0.2)
-		(layer "In1.Cu")
-		(net "CAN-")
-	)
-	(segment
-		(start 57.230492 101.503883)
-		(end 58.484375 100.25)
-		(width 0.2)
+		(start 127.86 99.42)
+		(end 129.71 101.27)
+		(width 0.12)
 		(layer "In1.Cu")
 		(net "CAN-")
 	)
 	(segment
-		(start 83.603554 99.5)
-		(end 127.94 99.5)
-		(width 0.2)
+		(start 83.336986 100.21)
+		(end 84.126986 99.42)
+		(width 0.12)
 		(layer "In1.Cu")
 		(net "CAN-")
