File: KiCad_PDM/KiCad_PDM.recovered.2026-07-28_175800.kicad_pcb (KiCad board)
At the start: 4 copper layers, 100 x 175 mm, 329 parts, among them J1 Conn_02x16_Top_Bottom, J2 6437288-1, J3 T66145145-1500, U1 74HC27D, U10 INA180A3IDBVR, U11 2N7002, U12 NSG2000, U13 OSP80N03T, U14 2N7002, U15 INA180A3IDBVR, U16 2N7002, U17 NSG2000, U18 OSP80N03T, U19 2N7002, U2 74HC27D, U20 INA180A3IDBVR, U21 2N7002, U22 NSG2000, U23 OSP80N03T, U24 2N7002, U25 INA180A3IDBVR, U26 2N7002, U27 NSG2000, U28 OSP80N03T, U29 2N7002, U3 74HC27D, U30 INA180A3IDBVR, U31 2N7002, U32 NSG2000, U33 OSP80N03T, U34 2N7002, U35 INA180A3IDBVR, U36 2N7002, U37 NSG2000, U38 OSP80N03T, U39 2N7002, U4 74HC27D, U40 INA180A3IDBVR, U41 2N7002, U42 NSG2000, U43 OSP80N03T, U44 2N7002, U45 INA180A3IDBVR, U46 2N7002, U47 NSG2000, U48 OSP80N03T, U49 2N7002, U5 KF33BDT-TR, U50 INA180A3IDBVR, U51 2N7002, U52 NSG2000, U53 OSP80N03T, U54 2N7002, U55 INA180A3IDBVR, U6 2N7002, U7 NSG2000, U8 OSP80N03T, U9 2N7002

Commit message: fixed CAN trace routing (diff pair), reduced digital signal trace size to 0.2mm
Parts:
- moved R50 7.60 mm to (97.0, 109.0)
- moved R51 6.10 mm to (102.0, 112.5), turned to 90 degrees
Connections:
- J1 pad 12: Aux3 -> unconnected-(J1-Pin_12-Pad12)
- J1 pad 13: Aux6 -> Aux3
- J1 pad 16: Aux2 -> Aux4
- J1 pad 19: Aux1 -> Aux6
- J1 pad 20: unconnected-(J1-Pin_20-Pad20) -> Aux1
- J1 pad 21: Aux5 -> Aux2
- J1 pad 23: Aux4 -> Aux5
- J2 pad 11: Aux4 -> Aux5
- J2 pad 12: Aux5 -> Aux2
- J2 pad 15: Aux6 -> Aux4
- J2 pad 6: Aux2 -> Aux6
Routing:
- net Aux4: track 80.9 -> 0.00 mm
- net Aux3: track 80.5 -> 0.00 mm
- net Aux5: track 78.9 -> 0.00 mm
- net Aux6: track 77.9 -> 0.00 mm
- net Aux2: track 77.7 -> 0.00 mm
- net Aux1: track 75.1 -> 0.00 mm
- net CS2: track 41.1 -> 0.00 mm, vias 1 -> 0
- net +3.3V: track 839.7 -> 803.6 mm, vias 21 -> 20
- net +BATT: track 253.1 -> 220.3 mm, vias 36 -> 37
- net Net-(C19-Pad2): track 38.6 -> 8.50 mm, vias 2 -> 0
- net Ch10_MCU: track 126.3 -> 116.0 mm
- net CS4: track 61.4 -> 52.7 mm
- net Ch8_MCU: track 116.6 -> 108.7 mm
- net /Ch3/Gate: track 9.09 -> 5.08 mm
- net Net-(U18-Gate): track 10.4 -> 6.90 mm
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