File: KiCad_PDM/KiCad_PDM.kicad_sch (KiCad schematic)
At the start: 69 parts, among them J1 Conn_02x16_Top_Bottom, J2 6437288-1, J3 T66145145-1500, U1 74HC27D, U2 74HC27D, U3 74HC27D, U4 74HC27D, U5 KF33BDT-TR

Commit message: added production files (gerbers, BOM, 3D models)
Parts:
- C57, C58: value C_Polarized -> 470uF
Changed lines of the file:
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@@
 		(in_pos_files yes)
 		(dnp no)
-		(fields_autoplaced yes)
 		(property "Reference" "C58"
-			(at 181.61 220.0909 0)
+			(at 181.61 220.98 0)
 			(show_name no)
 			(do_not_autoplace no)
@@
 			)
 		)
-		(property "Value" "C_Polarized"
-			(at 181.61 222.6309 0)
+		(property "Value" "470uF"
+			(at 181.61 223.52 0)
 			(show_name no)
 			(do_not_autoplace no)
@@
 		(in_pos_files yes)
 		(dnp no)
-		(fields_autoplaced yes)
 		(property "Reference" "C57"
-			(at 156.21 220.0909 0)
+			(at 156.21 220.98 0)
 			(show_name no)
 			(do_not_autoplace no)
@@
 			)
 		)
-		(property "Value" "C_Polarized"
-			(at 156.21 222.6309 0)
+		(property "Value" "470uF"
+			(at 156.21 223.52 0)
 			(show_name no)
 			(do_not_autoplace no)
