File: Controller/STM32 V2/STM32 V2.kicad_pcb (KiCad board)
At the start: 4 copper layers, 100 x 40 mm, 58 parts, among them J1 Conn_01x07, J3 Conn_02x16_Top_Bottom, SW1 SW_Push, SW2 SW_SPDT, U1 STM32G474RCT6, U2 SN65

Commit message: added new controller board (moved pinouts to match PDM, fixed CAN trace)
Parts:
- added R25: 120, Resistor_SMD:R_0805_2012Metric_Pad1.20x1.40mm_HandSolder, F.Cu at (176.6, 95.9)
- moved R19 72.8 mm to (124.8, 93.4)
- moved R12 72.8 mm to (124.8, 97.9)
- moved JP6 72.5 mm to (128.7, 93.9)
- moved R17 64.1 mm to (124.8, 102.4)
- moved R10 64.1 mm to (124.8, 106.9)
- moved JP4 63.3 mm to (128.7, 102.9)
- moved R1 57.5 mm to (124.8, 117.0)
- moved JP1 55.9 mm to (128.7, 112.6)
- moved R7 52.8 mm to (124.8, 112.2), turned to 90 degrees
- moved C17 42.3 mm to (168.5, 100.2), turned to 180 degrees
- moved U2 37.8 mm to (170.2, 95.9)
- moved JP3 19.9 mm to (199.2, 105.4)
- moved R3 19.9 mm to (195.6, 105.9)
- moved R9 19.9 mm to (195.6, 101.2)
- moved D1 15.1 mm to (184.5, 88.7)
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Connections:
- D1 pad 1: Net-(D1-K) -> Led1
- D1 pad 2: Led1 -> Net-(D1-A)
- D2 pad 1: Net-(D2-K) -> Led2
- D2 pad 2: Led2 -> Net-(D2-A)
- D3 pad 1: Net-(D3-K) -> Led3
- D3 pad 2: Led3 -> Net-(D3-A)
- J3 pad 12: unconnected-(J3-Pin_12-Pad12) -> Aux3
- J3 pad 13: Can_Lo -> Aux6
- J3 pad 15: Aux6 -> Can-
- J3 pad 16: Aux4 -> Aux2
- J3 pad 17: +BATT -> Can+
- J3 pad 18: Aux3 -> +BATT
- J3 pad 20: Aux2 -> unconnected-(J3-Pin_20-Pad20)
- J3 pad 23: Can_Hi -> Aux4
- R20 pad 1: Net-(D1-K) -> Net-(D1-A)
- R21 pad 1: Net-(D2-K) -> Net-(D2-A)
- R22 pad 1: Net-(D3-K) -> Net-(D3-A)
- U2 pad 6: Can_Lo -> Can-
- U2 pad 7: Can_Hi -> Can+
Routing:
- net +3.3V: track 325.2 -> 217.5 mm
- net Can+: track 0.00 -> 107.2 mm
- net Can-: track 0.00 -> 107.2 mm
- net Can_Hi: track 57.8 -> 0.00 mm, vias 1 -> 0
- net Aux3: track 32.7 -> 69.4 mm, vias 0 -> 1
- net Net-(JP4-C): track 55.8 -> 20.9 mm
- net Can_Lo: track 34.3 -> 0.00 mm, vias 2 -> 0
- net Aux6: track 77.6 -> 43.6 mm, vias 0 -> 1
- net CS5: track 22.1 -> 50.4 mm
- net /RX: track 38.7 -> 12.2 mm, vias 2 -> 0
- net Net-(JP6-C): track 58.1 -> 32.5 mm
- net Led3: track 24.5 -> 49.7 mm
- net Net-(U1-PA12): track 33.7 -> 9.06 mm, vias 2 -> 0
- net Aux4: track 71.1 -> 47.7 mm, vias 0 -> 1
- net Net-(JP3-C): track 44.1 -> 67.2 mm, vias 2 -> 0
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Other:
- board text added: "3.3V"
- board text added: "3.3v"
- board text added: "Colliculi@26'"
- board text added: "GND"
- board text added: "RST"
- board text added: "RX"
- board text added: "SWCLK"
- board text added: "SWDIO"
- board text added: "TX"
