File: Controller/STM32 V2/STM32 V2.kicad_sch (KiCad schematic)
At the start: 58 parts, among them J1 Conn_01x07, J3 Conn_02x16_Top_Bottom, SW1 SW_Push, SW2 SW_SPDT, U1 STM32G474RCT6, U2 SN65

Commit message: added new controller board (moved pinouts to match PDM, fixed CAN trace)
Parts:
- added R25: 120, Resistor_SMD:R_0805_2012Metric_Pad1.20x1.40mm_HandSolder, symbol Device:R
Connections:
- net +BATT: now also J3.18 (Pin_18); no longer J3.17 (Pin_17)
- net Aux2: now also J3.16 (Pin_16); no longer J3.20 (Pin_20)
- net Aux3: now also J3.12 (Pin_12); no longer J3.18 (Pin_18)
- net Aux4: now also J3.23 (Pin_23); no longer J3.16 (Pin_16)
- net Aux6: now also J3.13 (Pin_13); no longer J3.15 (Pin_15)
- net Led1: now also D1.1 (K); no longer D1.2 (A)
- net Led2: now also D2.1 (K); no longer D2.2 (A)
- net Led3: now also D3.1 (K); no longer D3.2 (A)
- net at R21.1: now also D2.2 (A); no longer D2.1 (K)
- net at R20.1: now also D1.2 (A); no longer D1.1 (K)
- net at R22.1: now also D3.2 (A); no longer D3.1 (K)
- net Can_Hi renamed Can+
- net Can+: now also J3.17 (Pin_17), R25.2; no longer J3.23 (Pin_23)
- net Can_Lo renamed Can-
- net Can-: now also J3.15 (Pin_15), R25.1; no longer J3.13 (Pin_13)
Other:
- moved on the sheet: C17, D1, D2, D3
